File: STM32G491.kicad_pcb (KiCad board)
At the start: 2 copper layers, 59 x 47.2 mm, 36 parts, among them IC1 TPD6E004RSER, J1 Conn_02x10_Odd_Even, J2 Conn_02x10_Odd_Even

Commit message: Agregar PNGS
Connections:
- IC1 pad 3: Net-(IC1-Pad3) -> /USB_D-
Routing:
- net GND: vias 70 -> 71
Other:
- board size 59 x 47.2 mm -> 58.2 x 44.2 mm
